Commit message: added drone sensors: thermal camera and ouster

File: rotors_description/urdf/component_snippets.xacro (robot description, xacro)
@@ -30,4 +30,58 @@
 	<waitToRecordBag>${wait_to_record_bag}</waitToRecordBag>
       </plugin>
+    </gazebo>
+  </xacro:macro>
+<!-- Macro to add Hokuyo range sensor -->
+<xacro:macro name="hokuyo_lidar" params="namespace parent_link">
+    <link name="${namespace}/hokuyo_link">
+      <inertial>
+         <mass value="0.01" />
+         <inertia ixx="1e-6" ixy="0.0" ixz="0.0" iyy="1e-6" iyz="0.0" izz="1e-6" />
+      </inertial>
+      <visual name="visual">
+        <geometry>
+          <mesh filename="package://rotors_description/meshes/hokuyo.dae" />
+        </geometry>
+      </visual>
+     </link>
+     <joint name="laser" type="fixed">
+      <parent link="${parent_link}" />
+      <child link="${namespace}/hokuyo_link" />
+      <origin xyz="0 0 0.05" rpy="0 0 0" />
+    </joint>
+    <gazebo reference="${namespace}/hokuyo_link">
+    <sensor type="gpu_ray" name="head_hokuyo_sensor">
+      <pose>0 0 0 0 0 0</pose>
+      <visualize>false</visualize>
+      <update_rate>40</update_rate>
+      <ray>
+        <scan>
+          <horizontal>
+            <samples>720</samples>
+            <resolution>1</resolution>
+            <min_angle>-2.35619</min_angle>
+            <max_angle>2.35619</max_angle>
+          </horizontal>
+        </scan>
+        <range>
+          <min>0.10</min>
+          <max>30.0</max>
+          <resolution>0.01</resolution>
+        </range>
+        <noise>
+          <type>gaussian</type>
+          <!-- Noise parameters based on published spec for Hokuyo laser
+               achieving "+-30mm" accuracy at range < 10m.  A mean of 0.0m and
+               stddev of 0.01m will put 99.7% of samples within 0.03m of the true
+               reading. -->
+          <mean>0.0</mean>
+          <stddev>0.01</stddev>
+        </noise>
+      </ray>
+      <plugin name="gazebo_ros_head_hokuyo_controller" filename="libgazebo_ros_gpu_laser.so">
+        <topicName>/drone11/scan</topicName>
+        <frameName>hokuyo_link</frameName>
+      </plugin>
+    </sensor>
     </gazebo>
   </xacro:macro>
@@ -109,4 +163,153 @@
         </plugin>
       </sensor>
+    </gazebo>
+  </xacro:macro>
+    <!-- Macro to add a thermal camera. -->
+  <xacro:macro name="thermal_camera_macro"
+    params="namespace parent_link camera_suffix ">
+    <link name="${namespace}/thermal_camera_${camera_suffix}_link">
+      <collision>
+        <origin xyz="0.10 0 0.425554" rpy="0 0 0"/>
+        <geometry>
+          <cylinder radius="0.01" length="0.006"/>
+        </geometry>
+      </collision>
+      <inertial>
+        <!--<mass value="0.1" />
+        <origin xyz="0 0 0" rpy="0 0 0" />
+        <inertia ixx="0.0000036" ixy="0" ixz="0" iyy="0.0000036" iyz="0" izz="0.0000067" />-->
+        <mass value="1e-5" />
+        <origin xyz="0 0 0" rpy="0 0 0" />
+        <inertia ixx="1e-6" ixy="0" ixz="0" iyy="1e-6" iyz="0" izz="1e-6" />
+      </inertial>
+    </link>
+    <joint name="${namespace}/thermal_camera_${camera_suffix}_joint" type="fixed">
+      <origin xyz="0 0 -0.5" rpy="0 0 0"/>
+      <axis xyz="1 0 0" />
+      <parent link="${parent_link}" />
+      <child link="${namespace}/thermal_camera_${camera_suffix}_link" />
+    </joint>
+    <link name="${namespace}/thermal_camera_${camera_suffix}_optical_link" />
+    <joint name="${namespace}/thermal_camera_${camera_suffix}_optical_joint" type="fixed" >
+      <origin xyz="0 0 0" rpy="${-pi/2} 0 ${-pi/2}" />
+      <parent link="${namespace}/thermal_camera_${camera_suffix}_link" />
+      <child link="${namespace}/thermal_camera_${camera_suffix}_optical_link" />
+    </joint>
+    <gazebo reference="${namespace}/thermal_camera_${camera_suffix}_link">
+      <sensor type="camera" name="${namespace}_thermal_camera_${camera_suffix}">
+        <update_rate>30</update_rate>
+        <camera name="head">
+<!--           <horizontal_fov>${horizontal_fov}</horizontal_fov> -->
+          <image>
+            <format>R8G8B8</format>
+            <width>186</width>
+            <height>100</height>
+          </image>
+          <clip>
+            <near>0.1</near>
+            <far>300</far>
+          </clip>
+        </camera>
+        <plugin name="${namespace}_thermal_camera_${camera_suffix}_controller" filename="libgazebo_ros_thermal_camera.so">
+          <robotNamespace>${namespace}</robotNamespace>
+          <cameraName>thermal_camera_${camera_suffix}</cameraName>
+          <frameName>thermal_camera_${camera_suffix}_link</frameName>
+          <alwaysOn>true</alwaysOn>
+          <updateRate>10</updateRate>
+          <!--<imageTopicName>${namespace}/thermal_camera/image_raw</imageTopicName>
+          <cameraInfoTopicName>${namespace}/thermal_camera/camera_info</cameraInfoTopicName>-->
+          <imageTopicName>image_raw</imageTopicName>
+          <cameraInfoTopicName>camera_info</cameraInfoTopicName>
+        </plugin>
+      </sensor>
+    </gazebo>
+  </xacro:macro>
+  <!-- Macro to add ouster lidar -->
+<xacro:macro name="ouster_lidar" params="namespace parent_link">
+    <link name="${namespace}/ouster_link">
+      <inertial>
+         <!--<mass value="0.1" />
+         <inertia ixx="0.000090623" ixy="0.0" ixz="0.0" iyy="0.000090623" iyz="0.0" izz="0.000091036" /> -->
+         <mass value="0.01" />
+         <inertia ixx="1e-6" ixy="0.0" ixz="0.0" iyy="1e-6" iyz="0.0" izz="1e-6" />
+      </inertial>
+      <!--<collision>
+        <origin xyz="-0.15 0 0.6462" rpy="0 0 0"/>
+        <geometry>
+          <cylinder radius="0.04267" length="0.07357"/>
+        </geometry>
+      </collision>-->
+     </link>
+      <link name="${namespace}/velodyne_base">
+      <inertial>
+         <!--<mass value="1.2" />
+         <inertia ixx="0.001087473" ixy="0.0" ixz="0.0" iyy="0.001087473" iyz="0.0" izz="0.001092437" /> -->
+         <mass value="0.01" />
+         <inertia ixx="1e-6" ixy="0.0" ixz="0.0" iyy="1e-6" iyz="0.0" izz="1e-6" />
+      </inertial>
+    <!--  <collision>
+        <origin xyz="-0.15 0 0.5801" rpy="0 0 0"/>
+        <geometry>
+          <cylinder radius="0.04267" length="0.05867"/>
+        </geometry>
+      </collision>-->
+     </link>
+    <joint type="fixed" name="joint">
+      <origin xyz="0 0 -0.036785" rpy="0 0 0" />
+      <parent link="${namespace}/velodyne_base" />
+      <child link="${namespace}/ouster_link" />
+      <axis>
+        <xyz>0 0 1</xyz>
+        <limit>
+          <lower>-10000000000000000</lower>
+          <upper>10000000000000000</upper>
+        </limit>
+      </axis>
+    </joint>
+    <joint type="fixed" name="fixed_velodyne">
+      <origin xyz="0 0 0" rpy="0 0 0" />
+      <parent link="${parent_link}" />
+      <child link="${namespace}/velodyne_base" />
+    </joint>
+    <gazebo reference="${namespace}/ouster_link">
+     <sensor type="ray" name="lase_scanr">
+      <pose>0 0 -0.004645 0 0 0</pose>
+      <visualize>false</visualize>
+      <update_rate>10</update_rate>
+      <ray>
+        <scan>
+            <horizontal>
+              <samples>512</samples>
+              <resolution>1</resolution>
+              <min_angle>-3.14159</min_angle>
+              <max_angle>3.14159</max_angle>
+            </horizontal>
+            <vertical>
+              <samples>16</samples>
+              <resolution>1</resolution>
+              <min_angle>-0.2897247</min_angle>
+              <max_angle>0.2897247</max_angle>
+            </vertical>
+        </scan>
+        <range>
+            <min>0.8</min>
+            <max>120</max>
+            <resolution>0.012</resolution>
+        </range>
+        <noise>
+            <type>gaussian</type>
+            <mean>0.0</mean>
+            <stddev>0.0</stddev>
+        </noise>
+      </ray>
+      <plugin name="${namespace}gazebo_ros_laser_controller" filename="libgazebo_ros_velodyne_laser.so">
+<!--           <topicName>${namespace}/os1_cloud_node/points</topicName> -->
+          <topicName>os1_cloud_node/points</topicName>
+          <frameName>os1_sensor</frameName>
+          <min_range>0.8</min_range>
+          <max_range>120.0</max_range>
+          <gaussianNoise>0.008</gaussianNoise>
+      </plugin>
+     </sensor>
     </gazebo>
   </xacro:macro>
@@ -497,40 +700,9 @@
     </gazebo>
   </xacro:macro>
-  <!-- Macro to add an air pressure sensor. -->
-  <xacro:macro name="pressure_sensor_plugin_macro"
-    params="namespace pressure_sensor_suffix parent_link pressure_topic
-      mass_pressure_sensor reference_altitude pressure_variance *inertia
-      *origin">
-    <!-- Pressure sensor link -->
-    <link name="${namespace}/pressure_sensor${pressure_sensor_suffix}_link">
-      <inertial>
-        <xacro:insert_block name="inertia" />
-        <mass value="${mass_pressure_sensor}" />  <!-- [kg] -->
-        <origin xyz="0 0 0" rpy="0 0 0" />
-      </inertial>
-    </link>
-    <!-- Pressure sensor joint -->
-    <joint name="${namespace}/pressure_sensor${pressure_sensor_suffix}_joint" type="revolute">
-      <xacro:insert_block name="origin" />
-      <parent link="${parent_link}" />
-      <child link="${namespace}/pressure_sensor${pressure_sensor_suffix}_link" />
-      <limit upper="0" lower="0" effort="0" velocity="0" />
-    </joint>
-    <gazebo>
-      <plugin filename="librotors_gazebo_pressure_plugin.so" name="rotors_gazebo_pressure_sensor${pressure_sensor_suffix}_plugin">
-        <robotNamespace>${namespace}</robotNamespace> <!-- (string, required): ros namespace in which the messages are published -->
-        <linkName>${namespace}/pressure_sensor${pressure_sensor_suffix}_link</linkName> <!-- (string, required): name of the body which holds the pressure sensor -->
-        <pressureTopic>${pressure_topic}</pressureTopic> <!-- (string): name of the sensor output topic and prefix of service names (defaults to 'air_pressure') -->
-        <referenceAltitude>${reference_altitude}</referenceAltitude> <!-- the initial altitude [m] -->
-        <pressureVariance>${pressure_variance}</pressureVariance> <!-- the air pressure variance [Pa^2] -->
-      </plugin>
-    </gazebo>
-  </xacro:macro>
   <!-- Macro to add the wind plugin. -->
   <xacro:macro name="wind_plugin_macro"
     params="namespace xyz_offset wind_direction wind_force_mean
       wind_gust_direction wind_gust_duration wind_gust_start
-      wind_gust_force_mean wind_speed_mean use_custom_static_wind_field
-      custom_wind_field_path">
+      wind_gust_force_mean wind_speed_mean">
     <gazebo>
       <plugin filename="librotors_gazebo_wind_plugin.so" name="wind_plugin">
@@ -546,6 +718,4 @@
         <windGustForceMean>${wind_gust_force_mean}</windGustForceMean> <!-- [N] -->
         <windSpeedMean>${wind_speed_mean}</windSpeedMean> <!-- [m/s] -->
-        <useCustomStaticWindField>${use_custom_static_wind_field}</useCustomStaticWindField>
-        <customWindFieldPath>${custom_wind_field_path}</customWindFieldPath> <!-- from ~/.ros -->
       </plugin>
     </gazebo>
@@ -865,17 +1035,4 @@
     </xacro:magnetometer_plugin_macro>
   </xacro:macro>
-  <xacro:macro name="default_pressure_sensor" params="namespace parent_link">
-    <xacro:pressure_sensor_plugin_macro
-      namespace="${namespace}"
-      pressure_sensor_suffix=""
-      parent_link="${parent_link}"
-      pressure_topic="air_pressure"
-      mass_pressure_sensor="0.015"
-      reference_altitude="500.0"
-      pressure_variance="0.0">
-      <inertia ixx="0.00001" ixy="0.0" ixz="0.0" iyy="0.00001" iyz="0.0" izz="0.00001" />
-      <origin xyz="0 0 0" rpy="0 0 0" />
-    </xacro:pressure_sensor_plugin_macro>
-  </xacro:macro>
   <xacro:macro name="default_mavlink_interface" params="namespace imu_sub_topic rotor_count">
     <xacro:mavlink_interface_macro

File: rotors_description/urdf/hummingbird_base.xacro (robot description, xacro)
@@ -39,3 +39,68 @@
       wait_to_record_bag="$(arg wait_to_record_bag)" />
   </xacro:if>
+  <gazebo reference="${namespace}/base_link">
+    <mu1>0.99</mu1>
+    <mu2>0.99</mu2>
+  </gazebo>
+<!--  <xacro:camera_macro
+    namespace="${namespace}"
+    parent_link="${namespace}/base_link"
+    camera_suffix="bottom"
+    frame_rate="50"
+    horizontal_fov="2.3"
+    image_width="640"
+    image_height="480"
+    image_format="R8G8B8"
+    min_distance="0.02"
+    max_distance="50"
+    noise_mean="0.0"
+    noise_stddev="0.007"
+    enable_visual="true">
+    <box size="0.002 0.005 0.005" />
+    <origin xyz="0 0 -0.05" rpy="0 1.57 0" />
+  </xacro:camera_macro>-->
+  <xacro:thermal_camera_macro
+    namespace="${namespace}"
+    parent_link="${namespace}/base_link"
+    camera_suffix="unique">
+  </xacro:thermal_camera_macro>
+  <xacro:ouster_lidar
+    namespace="${namespace}"
+    parent_link="${namespace}/base_link" >
+  </xacro:ouster_lidar>
+ <!--  <xacro:hokuyo_lidar
+    namespace="${namespace}"
+    parent_link="${namespace}/base_link" >
+  </xacro:hokuyo_lidar> -->
+<!--Contact sensor 1 Laser
+<joint name="contact_sensor_1_joint" type="fixed">
+    <axis xyz="0 1 0" />
+    <origin xyz="0 0 -0.1" rpy="0 0 0"/>
+    <parent link="${namespace}/base_link"/>
+    <child link="contact_sensor_1_link"/>
+  </joint>
+  <link name="contact_sensor_1_link">
+    <collision name="contact_sensor_collision_1">
+      <origin xyz="0 0 0" rpy="0 0 0"/>
+      <geometry>
+    	<box size="0.1 0.1 0.001"/>
+      </geometry>
+    </collision>
+    <visual name="contact_sensor_visual_1">
+      <origin xyz="0 0 0" rpy="0 0 0"/>
+      <geometry>
+    	<box size="0.01 0.01 0.001"/>
+      </geometry>
+    </visual>
+  </link>
+  <gazebo reference="contact_sensor_1_link">
+          <sensor name="contact_sensor_1" type="contact">
+		<plugin name="my_contact_plugin_1" filename="libgazebo_ros_bumper.so">
+			    <frameName>world</frameName>
+		</plugin>
+          <contact>
+            <collision>contact_sensor_collision_1_collision</collision>
+          </contact>
+      </sensor>
+  </gazebo>-->
 </robot>

Commit message: GPS integration

File: rotors_description/urdf/component_snippets.xacro (robot description, xacro)
@@ -28,5 +28,5 @@
         <frameId>${namespace}/base_link</frameId>
         <rotorVelocitySlowdownSim>${rotor_velocity_slowdown_sim}</rotorVelocitySlowdownSim>
-	<waitToRecordBag>${wait_to_record_bag}</waitToRecordBag>
+	      <waitToRecordBag>${wait_to_record_bag}</waitToRecordBag>
       </plugin>
     </gazebo>
@@ -304,5 +304,5 @@
       </ray>
       <plugin name="${namespace}gazebo_ros_laser_controller" filename="libgazebo_ros_velodyne_laser.so">
-<!--           <topicName>${namespace}/os1_cloud_node/points</topicName> -->
+          <!--<topicName>${namespace}/os1_cloud_node/points</topicName> -->
           <topicName>os1_cloud_node/points</topicName>
           <frameName>os1_sensor</frameName>
@@ -472,10 +472,10 @@
       <plugin name="mavlink_interface" filename="librotors_gazebo_mavlink_interface.so">
         <robotNamespace>${namespace}</robotNamespace>
-	<mavlinkControlSubTopic>${mavlink_sub_topic}</mavlinkControlSubTopic>
+	      <mavlinkControlSubTopic>${mavlink_sub_topic}</mavlinkControlSubTopic>
         <imuSubTopic>${imu_sub_topic}</imuSubTopic>
         <mavlinkHilSensorPubTopic>${mavlink_pub_topic}</mavlinkHilSensorPubTopic>
-	<motorSpeedsPubTopic>${motors_speeds_pub_topic}</motorSpeedsPubTopic>
-	<gpsUpdateFreq>${gps_update_freq}</gpsUpdateFreq> <!-- Frequency of HIL GPS messages [Hz] -->
-	<rotorCount>${rotor_count}</rotorCount>
+	      <motorSpeedsPubTopic>${motors_speeds_pub_topic}</motorSpeedsPubTopic>
+	      <gpsUpdateFreq>${gps_update_freq}</gpsUpdateFreq> <!-- Frequency of HIL GPS messages [Hz] -->
+	      <rotorCount>${rotor_count}</rotorCount>
         <!-- [Gauss] Below are the North, East, and Down components of the Earth's magnetic field at the reference location.
              The default reference location is Zurich (lat=+47.3667degN, lon=+8.5500degE, h=+500m, WGS84).

File: rotors_description/urdf/hummingbird_base.xacro (robot description, xacro)
@@ -69,4 +69,8 @@
     parent_link="${namespace}/base_link" >
   </xacro:ouster_lidar>
+  <xacro:default_gps
+    namespace="${namespace}"
+    parent_link="${namespace}/base_link" >
+  </xacro:default_gps>
  <!--  <xacro:hokuyo_lidar
     namespace="${namespace}"
@@ -74,5 +78,5 @@
   </xacro:hokuyo_lidar> -->
 <!--Contact sensor 1 Laser
-<joint name="contact_sensor_1_joint" type="fixed">
+  <joint name="contact_sensor_1_joint" type="fixed">
     <axis xyz="0 1 0" />
     <origin xyz="0 0 -0.1" rpy="0 0 0"/>

Commit message: Fixing GPS parameters

File: rotors_description/urdf/component_snippets.xacro (robot description, xacro)
@@ -213,6 +213,6 @@
         <plugin name="${namespace}_thermal_camera_${camera_suffix}_controller" filename="libgazebo_ros_thermal_camera.so">
           <robotNamespace>${namespace}</robotNamespace>
-          <cameraName>thermal_camera_${camera_suffix}</cameraName>
-          <frameName>thermal_camera_${camera_suffix}_link</frameName>
+          <cameraName>thermal_camera</cameraName>  <!--USING FOR DOMI: thermal_camera_${camera_suffix} -->
+          <frameName>thermal_camera_link</frameName> <!--USING FOR DOMI: thermal_camera_${camera_suffix}_link -->
           <alwaysOn>true</alwaysOn>
           <updateRate>10</updateRate>
@@ -225,7 +225,46 @@
     </gazebo>
   </xacro:macro>
+  <!-- Macro to add a GPS fix -->
+  <xacro:macro name="gps_fix_macro" params="namespace parent_link gps_suffix">
+    <link name="${namespace}/gps_fix_${gps_suffix}_link">
+      <!-- <collision>
+        <origin xyz="0.10 0 0.425554" rpy="0 0 0"/>
+        <geometry>
+          <cylinder radius="0.01" length="0.006"/>
+        </geometry>
+      </collision>      -->
+      <inertial>
+        <mass value="0.01" />
+        <!-- <origin xyz="0 0 0" rpy="0 0 0" /> -->
+        <inertia ixx="1e-6" ixy="0" ixz="0" iyy="1e-6" iyz="0" izz="1e-6" />
+      </inertial>
+    </link>
+    <joint name="${namespace}/gps_fix_${gps_suffix}_joint" type="fixed">
+      <origin xyz="0 0 0.5" rpy="0 0 0"/>
+      <!-- <axis xyz="1 0 0" /> -->
+      <parent link="${parent_link}" />
+      <child link="${namespace}/gps_fix_${gps_suffix}_link" />
+    </joint>
+    <gazebo reference="${namespace}/gps_fix_${gps_suffix}_link">
+      <sensor type="gps" name="gps_fix_${gps_suffix}">
+        <plugin name="${namespace}_gps_fix_dron_${gps_suffix}" filename="libgazebo_ros_gps.so">
+              <alwaysOn>true</alwaysOn>
+              <updateRate>5.0</updateRate>
+              <!-- <bodyName>base_link</bodyName> -->
+              <topicName>${namespace}/gps{gps_suffix}</topicName>
+              <frameId>${namespace}/base_link{gps_suffix}</frameId>
+              <robotBaseFrame>${namespace}/base_link{gps_suffix}</robotBaseFrame>
+              <velocityTopicName>${namespace}/gps_velocity{gps_suffix}</velocityTopicName>
+              <drift>5.0 5.0 5.0</drift>
+              <gaussianNoise>0.1 0.1 0.1</gaussianNoise>
+              <velocityDrift>0 0 0</velocityDrift>
+              <velocityGaussianNoise>0.1 0.1 0.1</velocityGaussianNoise>
+          </plugin>
+        </sensor>
+    </gazebo>
+  </xacro:macro>
   <!-- Macro to add ouster lidar -->
 <xacro:macro name="ouster_lidar" params="namespace parent_link">
-    <link name="${namespace}/ouster_link">
+    <link name="${namespace}/os1_sensor">
       <inertial>
          <!--<mass value="0.1" />
@@ -240,6 +279,6 @@
         </geometry>
       </collision>-->
-     </link>
-      <link name="${namespace}/velodyne_base">
+    </link>
+    <link name="${namespace}/velodyne_base">
       <inertial>
          <!--<mass value="1.2" />
@@ -254,9 +293,9 @@
         </geometry>
       </collision>-->
-     </link>
+    </link>
     <joint type="fixed" name="joint">
       <origin xyz="0 0 -0.036785" rpy="0 0 0" />
       <parent link="${namespace}/velodyne_base" />
-      <child link="${namespace}/ouster_link" />
+      <child link="${namespace}/os1_sensor" />
       <axis>
         <xyz>0 0 1</xyz>
@@ -272,6 +311,6 @@
       <child link="${namespace}/velodyne_base" />
     </joint>
-    <gazebo reference="${namespace}/ouster_link">
-     <sensor type="ray" name="lase_scanr">
+    <gazebo reference="${namespace}/os1_sensor">
+     <sensor type="ray" name="laser_scan">
       <pose>0 0 -0.004645 0 0 0</pose>
       <visualize>false</visualize>
@@ -485,5 +524,5 @@
         <referenceMagEast>${reference_magnetic_field_east}</referenceMagEast>
         <referenceMagDown>${reference_magnetic_field_down}</referenceMagDown>
-	<referenceLatitude>${reference_latitude}</referenceLatitude> <!-- the initial latitude [degrees [-90, 90]] -->
+	      <referenceLatitude>${reference_latitude}</referenceLatitude> <!-- the initial latitude [degrees [-90, 90]] -->
         <referenceLongitude>${reference_longitude}</referenceLongitude> <!-- the initial longitude [degrees [-180, 180]] -->
         <referenceAltitude>${reference_altitude}</referenceAltitude> <!-- the initial altitude [m] -->
@@ -652,5 +691,5 @@
         <plugin filename="librotors_gazebo_gps_plugin.so" name="rotors_gazebo_gps${gps_suffix}_plugin">
           <robotNamespace>${namespace}</robotNamespace> <!-- (string, required): ros namespace in which the messages are published -->
-          <linkName>${namespace}/gps${gps_suffix}_link</linkName> <!-- (string, required): name of the body which holds the GPS sensor -->
+          <linkName>${namespace}/base_link</linkName> <!-- (string, required): name of the body which holds the GPS sensor -->
           <gpsTopic>${gps_topic}</gpsTopic> <!-- (string): name of the sensor output topic and prefix of service names (defaults to 'gps') -->
           <groundSpeedTopic>${ground_speed_topic}</groundSpeedTopic> <!-- (string): name of the ground speed output topic (defaults to 'ground_speed') -->
@@ -1035,4 +1074,8 @@
     </xacro:magnetometer_plugin_macro>
   </xacro:macro>
+  <!-- DEFAULT VALUES OF REFERENCES -->
+  <!--reference_latitude="47.3667"
+      reference_longitude="8.5500"
+      reference_altitude="500.0" -->
   <xacro:macro name="default_mavlink_interface" params="namespace imu_sub_topic rotor_count">
     <xacro:mavlink_interface_macro
@@ -1047,7 +1090,7 @@
       reference_magnetic_field_east="0.00797"
       reference_magnetic_field_down="0.42817"
-      reference_latitude="47.3667"
-      reference_longitude="8.5500"
-      reference_altitude="500.0">
+      reference_latitude="49.9"
+      reference_longitude="8.9"
+      reference_altitude="0.0">
     </xacro:mavlink_interface_macro>
   </xacro:macro>

File: rotors_description/urdf/hummingbird_base.xacro (robot description, xacro)
@@ -69,7 +69,12 @@
     parent_link="${namespace}/base_link" >
   </xacro:ouster_lidar>
+  <!-- <xacro:gps_fix_macro
+    namespace="${namespace}"
+    parent_link="${namespace}/base_link"
+    gps_suffix="fix">
+  </xacro:gps_fix_macro>   -->
   <xacro:default_gps
     namespace="${namespace}"
-    parent_link="${namespace}/base_link" >
+    parent_link="${namespace}/base_link">
   </xacro:default_gps>
  <!--  <xacro:hokuyo_lidar
