Commit message: Fixed GPS for MBZIRC system

File: rotors_description/urdf/component_snippets.xacro (robot description, xacro)
@@ -226,40 +226,33 @@
   </xacro:macro>
   <!-- Macro to add a GPS fix -->
-  <xacro:macro name="gps_fix_macro" params="namespace parent_link gps_suffix">
-    <link name="${namespace}/gps_fix_${gps_suffix}_link">
-      <!-- <collision>
-        <origin xyz="0.10 0 0.425554" rpy="0 0 0"/>
-        <geometry>
-          <cylinder radius="0.01" length="0.006"/>
-        </geometry>
-      </collision>      -->
+  <xacro:macro name="gps_fix_macro" params="namespace parent_link">
+    <link name="${namespace}/gps_fix_link">
       <inertial>
         <mass value="0.01" />
-        <!-- <origin xyz="0 0 0" rpy="0 0 0" /> -->
         <inertia ixx="1e-6" ixy="0" ixz="0" iyy="1e-6" iyz="0" izz="1e-6" />
       </inertial>
     </link>
-    <joint name="${namespace}/gps_fix_${gps_suffix}_joint" type="fixed">
-      <origin xyz="0 0 0.5" rpy="0 0 0"/>
-      <!-- <axis xyz="1 0 0" /> -->
-      <parent link="${parent_link}" />
-      <child link="${namespace}/gps_fix_${gps_suffix}_link" />
-    </joint>
-    <gazebo reference="${namespace}/gps_fix_${gps_suffix}_link">
-      <sensor type="gps" name="gps_fix_${gps_suffix}">
-        <plugin name="${namespace}_gps_fix_dron_${gps_suffix}" filename="libgazebo_ros_gps.so">
+    <joint name="${namespace}/gps_fix_joint" type="fixed">
+      <origin xyz="0 0 0.05" rpy="0 0 0"/>
+      <parent link="${parent_link}" />
+      <child link="${namespace}/gps_fix_link" />
+    </joint>
+    <gazebo >
+              <plugin name="${namespace}_gps_fix_dron" filename="libplugin_gazebo_ros_gps.so">
+              <updateRate>5.0</updateRate>
+              <bodyName>${namespace}/base_link</bodyName>
               <alwaysOn>true</alwaysOn>
-              <updateRate>5.0</updateRate>
-              <!-- <bodyName>base_link</bodyName> -->
-              <topicName>${namespace}/gps{gps_suffix}</topicName>
-              <frameId>${namespace}/base_link{gps_suffix}</frameId>
-              <robotBaseFrame>${namespace}/base_link{gps_suffix}</robotBaseFrame>
-              <velocityTopicName>${namespace}/gps_velocity{gps_suffix}</velocityTopicName>
-              <drift>5.0 5.0 5.0</drift>
+              <robotBaseFrame>${namespace}/base_link</robotBaseFrame>
+              <!-- <frameId>${namespace}/base_link</frameId> -->
+              <topicName>gps</topicName>
+              <velocityTopicName>gps_velocity</velocityTopicName>
               <gaussianNoise>0.1 0.1 0.1</gaussianNoise>
               <velocityDrift>0 0 0</velocityDrift>
               <velocityGaussianNoise>0.1 0.1 0.1</velocityGaussianNoise>
+              <referenceLatitude>49.9</referenceLatitude>
+              <referenceLongitude>8.9</referenceLongitude>
+              <referenceHeading>0</referenceHeading>
+              <referenceAltitude>0</referenceAltitude>
           </plugin>
-        </sensor>
     </gazebo>
   </xacro:macro>

File: rotors_description/urdf/hummingbird_base.xacro (robot description, xacro)
@@ -69,13 +69,12 @@
     parent_link="${namespace}/base_link" >
   </xacro:ouster_lidar>
-  <!-- <xacro:gps_fix_macro
-    namespace="${namespace}"
-    parent_link="${namespace}/base_link"
-    gps_suffix="fix">
-  </xacro:gps_fix_macro>   -->
-  <xacro:default_gps
+  <xacro:gps_fix_macro
     namespace="${namespace}"
     parent_link="${namespace}/base_link">
-  </xacro:default_gps>
+  </xacro:gps_fix_macro>
+  <!-- <xacro:default_gps
+    namespace="${namespace}"
+    parent_link="${namespace}/base_link">
+  </xacro:default_gps>   -->
  <!--  <xacro:hokuyo_lidar
     namespace="${namespace}"

Commit message: Fixed GPS for MBZIRC system

File: rotors_description/urdf/component_snippets.xacro (robot description, xacro)
@@ -17,5 +17,5 @@
 -->
 <robot xmlns:xacro="http://ros.org/wiki/xacro">
-  <xacro:property name="pi" value="3.14159265359" />
+  <xacro:property name="M_PI" value="3.14159265359" />
   <!-- Macro to add logging to a bag file. -->
   <xacro:macro name="bag_plugin_macro"
@@ -163,185 +163,4 @@
         </plugin>
       </sensor>
-    </gazebo>
-  </xacro:macro>
-    <!-- Macro to add a thermal camera. -->
-  <xacro:macro name="thermal_camera_macro"
-    params="namespace parent_link camera_suffix ">
-    <link name="${namespace}/thermal_camera_${camera_suffix}_link">
-      <collision>
-        <origin xyz="0.10 0 0.425554" rpy="0 0 0"/>
-        <geometry>
-          <cylinder radius="0.01" length="0.006"/>
-        </geometry>
-      </collision>
-      <inertial>
-        <!--<mass value="0.1" />
-        <origin xyz="0 0 0" rpy="0 0 0" />
-        <inertia ixx="0.0000036" ixy="0" ixz="0" iyy="0.0000036" iyz="0" izz="0.0000067" />-->
-        <mass value="1e-5" />
-        <origin xyz="0 0 0" rpy="0 0 0" />
-        <inertia ixx="1e-6" ixy="0" ixz="0" iyy="1e-6" iyz="0" izz="1e-6" />
-      </inertial>
-    </link>
-    <joint name="${namespace}/thermal_camera_${camera_suffix}_joint" type="fixed">
-      <origin xyz="0 0 -0.5" rpy="0 0 0"/>
-      <axis xyz="1 0 0" />
-      <parent link="${parent_link}" />
-      <child link="${namespace}/thermal_camera_${camera_suffix}_link" />
-    </joint>
-    <link name="${namespace}/thermal_camera_${camera_suffix}_optical_link" />
-    <joint name="${namespace}/thermal_camera_${camera_suffix}_optical_joint" type="fixed" >
-      <origin xyz="0 0 0" rpy="${-pi/2} 0 ${-pi/2}" />
-      <parent link="${namespace}/thermal_camera_${camera_suffix}_link" />
-      <child link="${namespace}/thermal_camera_${camera_suffix}_optical_link" />
-    </joint>
-    <gazebo reference="${namespace}/thermal_camera_${camera_suffix}_link">
-      <sensor type="camera" name="${namespace}_thermal_camera_${camera_suffix}">
-        <update_rate>30</update_rate>
-        <camera name="head">
-<!--           <horizontal_fov>${horizontal_fov}</horizontal_fov> -->
-          <image>
-            <format>R8G8B8</format>
-            <width>186</width>
-            <height>100</height>
-          </image>
-          <clip>
-            <near>0.1</near>
-            <far>300</far>
-          </clip>
-        </camera>
-        <plugin name="${namespace}_thermal_camera_${camera_suffix}_controller" filename="libgazebo_ros_thermal_camera.so">
-          <robotNamespace>${namespace}</robotNamespace>
-          <cameraName>thermal_camera</cameraName>  <!--USING FOR DOMI: thermal_camera_${camera_suffix} -->
-          <frameName>thermal_camera_link</frameName> <!--USING FOR DOMI: thermal_camera_${camera_suffix}_link -->
-          <alwaysOn>true</alwaysOn>
-          <updateRate>10</updateRate>
-          <!--<imageTopicName>${namespace}/thermal_camera/image_raw</imageTopicName>
-          <cameraInfoTopicName>${namespace}/thermal_camera/camera_info</cameraInfoTopicName>-->
-          <imageTopicName>image_raw</imageTopicName>
-          <cameraInfoTopicName>camera_info</cameraInfoTopicName>
-        </plugin>
-      </sensor>
-    </gazebo>
-  </xacro:macro>
-  <!-- Macro to add a GPS fix -->
-  <xacro:macro name="gps_fix_macro" params="namespace parent_link">
-    <link name="${namespace}/gps_fix_link">
-      <inertial>
-        <mass value="0.01" />
-        <inertia ixx="1e-6" ixy="0" ixz="0" iyy="1e-6" iyz="0" izz="1e-6" />
-      </inertial>
-    </link>
-    <joint name="${namespace}/gps_fix_joint" type="fixed">
-      <origin xyz="0 0 0.05" rpy="0 0 0"/>
-      <parent link="${parent_link}" />
-      <child link="${namespace}/gps_fix_link" />
-    </joint>
-    <gazebo >
-              <plugin name="${namespace}_gps_fix_dron" filename="libplugin_gazebo_ros_gps.so">
-              <updateRate>5.0</updateRate>
-              <bodyName>${namespace}/base_link</bodyName>
-              <alwaysOn>true</alwaysOn>
-              <robotBaseFrame>${namespace}/base_link</robotBaseFrame>
-              <!-- <frameId>${namespace}/base_link</frameId> -->
-              <topicName>gps</topicName>
-              <velocityTopicName>gps_velocity</velocityTopicName>
-              <gaussianNoise>0.1 0.1 0.1</gaussianNoise>
-              <velocityDrift>0 0 0</velocityDrift>
-              <velocityGaussianNoise>0.1 0.1 0.1</velocityGaussianNoise>
-              <referenceLatitude>49.9</referenceLatitude>
-              <referenceLongitude>8.9</referenceLongitude>
-              <referenceHeading>0</referenceHeading>
-              <referenceAltitude>0</referenceAltitude>
-          </plugin>
-    </gazebo>
-  </xacro:macro>
-  <!-- Macro to add ouster lidar -->
-<xacro:macro name="ouster_lidar" params="namespace parent_link">
-    <link name="${namespace}/os1_sensor">
-      <inertial>
-         <!--<mass value="0.1" />
-         <inertia ixx="0.000090623" ixy="0.0" ixz="0.0" iyy="0.000090623" iyz="0.0" izz="0.000091036" /> -->
-         <mass value="0.01" />
-         <inertia ixx="1e-6" ixy="0.0" ixz="0.0" iyy="1e-6" iyz="0.0" izz="1e-6" />
-      </inertial>
-      <!--<collision>
-        <origin xyz="-0.15 0 0.6462" rpy="0 0 0"/>
-        <geometry>
-          <cylinder radius="0.04267" length="0.07357"/>
-        </geometry>
-      </collision>-->
-    </link>
-    <link name="${namespace}/velodyne_base">
-      <inertial>
-         <!--<mass value="1.2" />
-         <inertia ixx="0.001087473" ixy="0.0" ixz="0.0" iyy="0.001087473" iyz="0.0" izz="0.001092437" /> -->
-         <mass value="0.01" />
-         <inertia ixx="1e-6" ixy="0.0" ixz="0.0" iyy="1e-6" iyz="0.0" izz="1e-6" />
-      </inertial>
-    <!--  <collision>
-        <origin xyz="-0.15 0 0.5801" rpy="0 0 0"/>
-        <geometry>
-          <cylinder radius="0.04267" length="0.05867"/>
-        </geometry>
-      </collision>-->
-    </link>
-    <joint type="fixed" name="joint">
-      <origin xyz="0 0 -0.036785" rpy="0 0 0" />
-      <parent link="${namespace}/velodyne_base" />
-      <child link="${namespace}/os1_sensor" />
-      <axis>
-        <xyz>0 0 1</xyz>
-        <limit>
-          <lower>-10000000000000000</lower>
-          <upper>10000000000000000</upper>
-        </limit>
-      </axis>
-    </joint>
-    <joint type="fixed" name="fixed_velodyne">
-      <origin xyz="0 0 0" rpy="0 0 0" />
-      <parent link="${parent_link}" />
-      <child link="${namespace}/velodyne_base" />
-    </joint>
-    <gazebo reference="${namespace}/os1_sensor">
-     <sensor type="ray" name="laser_scan">
-      <pose>0 0 -0.004645 0 0 0</pose>
-      <visualize>false</visualize>
-      <update_rate>10</update_rate>
-      <ray>
-        <scan>
-            <horizontal>
-              <samples>512</samples>
-              <resolution>1</resolution>
-              <min_angle>-3.14159</min_angle>
-              <max_angle>3.14159</max_angle>
-            </horizontal>
-            <vertical>
-              <samples>16</samples>
-              <resolution>1</resolution>
-              <min_angle>-0.2897247</min_angle>
-              <max_angle>0.2897247</max_angle>
-            </vertical>
-        </scan>
-        <range>
-            <min>0.8</min>
-            <max>120</max>
-            <resolution>0.012</resolution>
-        </range>
-        <noise>
-            <type>gaussian</type>
-            <mean>0.0</mean>
-            <stddev>0.0</stddev>
-        </noise>
-      </ray>
-      <plugin name="${namespace}gazebo_ros_laser_controller" filename="libgazebo_ros_velodyne_laser.so">
-          <!--<topicName>${namespace}/os1_cloud_node/points</topicName> -->
-          <topicName>os1_cloud_node/points</topicName>
-          <frameName>os1_sensor</frameName>
-          <min_range>0.8</min_range>
-          <max_range>120.0</max_range>
-          <gaussianNoise>0.008</gaussianNoise>
-      </plugin>
-     </sensor>
     </gazebo>
   </xacro:macro>

File: rotors_description/urdf/hummingbird_base.xacro (robot description, xacro)
@@ -18,4 +18,5 @@
 <robot name="hummingbird" xmlns:xacro="http://ros.org/wiki/xacro">
   <xacro:include filename="$(find rotors_description)/urdf/component_snippets.xacro" />
+  <xacro:include filename="$(find rotors_description)/urdf/component_mbzirc.xacro" />
   <!-- Instantiate hummingbird "mechanics" -->
   <xacro:include filename="$(find rotors_description)/urdf/hummingbird.xacro" />
