Commit message: Added tf plugin to FIREFLY DRON

File: rotors_description/urdf/component_mbzirc.xacro (robot description, xacro)
@@ -182,3 +182,11 @@
     </gazebo>
   </xacro:macro>
+  <xacro:macro name="gazebo_tf_plugin_macro" params="namespace">
+    <gazebo>
+      <plugin name="gazebo_tf_firefly_plugin" filename="libgazego_tf_firefly_plugin.so">
+        <robotNamespace>${namespace}</robotNamespace>
+        <updateRate>50.0</updateRate>
+      </plugin>
+    </gazebo>
+  </xacro:macro>
   </robot>

File: rotors_description/urdf/firefly_base.xacro (robot description, xacro)
@@ -18,4 +18,5 @@
 <robot name="firefly" xmlns:xacro="http://ros.org/wiki/xacro">
   <xacro:include filename="$(find rotors_description)/urdf/component_snippets.xacro" />
+  <xacro:include filename="$(find rotors_description)/urdf/component_mbzirc.xacro" />
   <!-- Instantiate firefly "mechanics" -->
   <xacro:include filename="$(find rotors_description)/urdf/firefly.xacro" />
@@ -33,4 +34,7 @@
     <xacro:ground_truth_imu_and_odometry namespace="${namespace}" parent_link="${namespace}/base_link" />
   </xacro:if>
+  <xacro:if value="$(arg pub_tf)">
+    <xacro:gazebo_tf_plugin_macro namespace="${namespace}"/>
+  </xacro:if>
   <xacro:if value="$(arg enable_logging)">
     <!-- Instantiate a logger -->

Commit message: added thermal camera looking down

File: rotors_description/urdf/component_mbzirc.xacro (robot description, xacro)
@@ -51,4 +51,64 @@
           <cameraName>thermal_camera</cameraName>  <!--USING FOR DOMI: thermal_camera_${camera_suffix} -->
           <frameName>thermal_camera_link</frameName> <!--USING FOR DOMI: thermal_camera_${camera_suffix}_link -->
+          <alwaysOn>true</alwaysOn>
+          <updateRate>10</updateRate>
+          <!--<imageTopicName>${namespace}/thermal_camera/image_raw</imageTopicName>
+          <cameraInfoTopicName>${namespace}/thermal_camera/camera_info</cameraInfoTopicName>-->
+          <imageTopicName>image_raw</imageTopicName>
+          <cameraInfoTopicName>camera_info</cameraInfoTopicName>
+        </plugin>
+      </sensor>
+    </gazebo>
+  </xacro:macro>
+    <!-- Macro to add a thermal camera looking down. -->
+  <xacro:macro name="thermal_camera_down_macro"
+    params="namespace parent_link camera_suffix ">
+    <link name="${namespace}/thermal_camera_down${camera_suffix}_link">
+      <!-- <collision>
+        <origin xyz="0.10 0 0.425554" rpy="0 0 0"/>
+        <geometry>
+          <cylinder radius="0.01" length="0.006"/>
+        </geometry>
+      </collision> -->
+      <inertial>
+        <!--<mass value="0.1" />
+        <origin xyz="0 0 0" rpy="0 0 0" />
+        <inertia ixx="0.0000036" ixy="0" ixz="0" iyy="0.0000036" iyz="0" izz="0.0000067" />-->
+        <mass value="1e-5" />
+        <origin xyz="0 0 0" rpy="0 0 0" />
+        <inertia ixx="1e-6" ixy="0" ixz="0" iyy="1e-6" iyz="0" izz="1e-6" />
+      </inertial>
+    </link>
+    <joint name="${namespace}/thermal_camera_down${camera_suffix}_joint" type="fixed">
+      <origin xyz="0 0 -0.5" rpy="0 ${pi/2} 0"/>
+      <axis xyz="1 0 0" />
+      <parent link="${parent_link}" />
+      <child link="${namespace}/thermal_camera_down${camera_suffix}_link" />
+    </joint>
+    <link name="${namespace}/thermal_camera_down${camera_suffix}_optical_link" />
+    <joint name="${namespace}/thermal_camera_down${camera_suffix}_optical_joint" type="fixed" >
+      <origin xyz="0 0 0" rpy="${-pi/2} 0 ${-pi/2}" />
+      <parent link="${namespace}/thermal_camera_down${camera_suffix}_link" />
+      <child link="${namespace}/thermal_camera_down${camera_suffix}_optical_link" />
+    </joint>
+    <gazebo reference="${namespace}/thermal_camera_down${camera_suffix}_link">
+      <sensor type="camera" name="${namespace}_thermal_camera_down${camera_suffix}">
+        <update_rate>30</update_rate>
+        <camera name="head">
+<!--           <horizontal_fov>${horizontal_fov}</horizontal_fov> -->
+          <image>
+            <format>R8G8B8</format>
+            <width>186</width>
+            <height>100</height>
+          </image>
+          <clip>
+            <near>0.1</near>
+            <far>300</far>
+          </clip>
+        </camera>
+        <plugin name="${namespace}_thermal_camera_down${camera_suffix}_controller" filename="libgazebo_ros_thermal_camera.so">
+          <robotNamespace>${namespace}</robotNamespace>
+          <cameraName>thermal_camera_down</cameraName>  <!--USING FOR DOMI: thermal_camera_${camera_suffix} -->
+          <frameName>thermal_camera_down_link</frameName> <!--USING FOR DOMI: thermal_camera_${camera_suffix}_link -->
           <alwaysOn>true</alwaysOn>
           <updateRate>10</updateRate>

File: rotors_description/urdf/firefly_base.xacro (robot description, xacro)
@@ -40,4 +40,7 @@
   <xacro:thermal_camera_macro namespace="${namespace}" parent_link="${namespace}/base_link" camera_suffix="unique">
   </xacro:thermal_camera_macro>
+  <!-- Adding thermal camera looking down -->
+  <xacro:thermal_camera_down_macro namespace="${namespace}" parent_link="${namespace}/base_link" camera_suffix="unique">
+  </xacro:thermal_camera_down_macro>
   <xacro:ouster_lidar namespace="${namespace}" parent_link="${namespace}/base_link">
   </xacro:ouster_lidar>

Commit message: migration to gazebo 9 and ros melodic.

File: rotors_description/urdf/component_mbzirc.xacro (robot description, xacro)
@@ -61,4 +61,64 @@
     </gazebo>
   </xacro:macro>
+    <!-- Macro to add a thermal camera looking down. -->
+  <xacro:macro name="thermal_camera_down_macro"
+    params="namespace parent_link camera_suffix ">
+    <link name="${namespace}/thermal_camera_down${camera_suffix}_link">
+      <!-- <collision>
+        <origin xyz="0.10 0 0.425554" rpy="0 0 0"/>
+        <geometry>
+          <cylinder radius="0.01" length="0.006"/>
+        </geometry>
+      </collision> -->
+      <inertial>
+        <!--<mass value="0.1" />
+        <origin xyz="0 0 0" rpy="0 0 0" />
+        <inertia ixx="0.0000036" ixy="0" ixz="0" iyy="0.0000036" iyz="0" izz="0.0000067" />-->
+        <mass value="1e-5" />
+        <origin xyz="0 0 0" rpy="0 0 0" />
+        <inertia ixx="1e-6" ixy="0" ixz="0" iyy="1e-6" iyz="0" izz="1e-6" />
+      </inertial>
+    </link>
+    <joint name="${namespace}/thermal_camera_down${camera_suffix}_joint" type="fixed">
+      <origin xyz="0 0 -0.5" rpy="0 ${pi/2} 0"/>
+      <axis xyz="1 0 0" />
+      <parent link="${parent_link}" />
+      <child link="${namespace}/thermal_camera_down${camera_suffix}_link" />
+    </joint>
+    <link name="${namespace}/thermal_camera_down${camera_suffix}_optical_link" />
+    <joint name="${namespace}/thermal_camera_down${camera_suffix}_optical_joint" type="fixed" >
+      <origin xyz="0 0 0" rpy="${-pi/2} 0 ${-pi/2}" />
+      <parent link="${namespace}/thermal_camera_down${camera_suffix}_link" />
+      <child link="${namespace}/thermal_camera_down${camera_suffix}_optical_link" />
+    </joint>
+    <gazebo reference="${namespace}/thermal_camera_down${camera_suffix}_link">
+      <sensor type="camera" name="${namespace}_thermal_camera_down${camera_suffix}">
+        <update_rate>30</update_rate>
+        <camera name="head">
+<!--           <horizontal_fov>${horizontal_fov}</horizontal_fov> -->
+          <image>
+            <format>R8G8B8</format>
+            <width>186</width>
+            <height>100</height>
+          </image>
+          <clip>
+            <near>0.1</near>
+            <far>300</far>
+          </clip>
+        </camera>
+        <plugin name="${namespace}_thermal_camera_down${camera_suffix}_controller" filename="libgazebo_ros_thermal_camera.so">
+          <robotNamespace>${namespace}</robotNamespace>
+          <cameraName>thermal_camera_down</cameraName>  <!--USING FOR DOMI: thermal_camera_${camera_suffix} -->
+          <frameName>thermal_camera_down_link</frameName> <!--USING FOR DOMI: thermal_camera_${camera_suffix}_link -->
+          <alwaysOn>true</alwaysOn>
+          <updateRate>10</updateRate>
+          <!--<imageTopicName>${namespace}/thermal_camera/image_raw</imageTopicName>
+          <cameraInfoTopicName>${namespace}/thermal_camera/camera_info</cameraInfoTopicName>-->
+          <imageTopicName>image_raw</imageTopicName>
+          <cameraInfoTopicName>camera_info</cameraInfoTopicName>
+        </plugin>
+      </sensor>
+    </gazebo>
+  </xacro:macro>
   <!-- Macro to add a GPS fix -->
   <xacro:macro name="gps_fix_macro" params="namespace parent_link">
@@ -83,7 +143,7 @@
               <topicName>gps</topicName>
               <velocityTopicName>gps_velocity</velocityTopicName>
-              <gaussianNoise>0.1 0.1 0.1</gaussianNoise>
+              <gaussianNoise>0.05 0.05 0.05</gaussianNoise>
               <velocityDrift>0 0 0</velocityDrift>
-              <velocityGaussianNoise>0.1 0.1 0.1</velocityGaussianNoise>
+              <velocityGaussianNoise>0.05 0.05 0.05</velocityGaussianNoise>
               <referenceLatitude>49.9</referenceLatitude>
               <referenceLongitude>8.9</referenceLongitude>
@@ -177,5 +237,5 @@
           <min_range>0.8</min_range>
           <max_range>120.0</max_range>
-          <gaussianNoise>0.008</gaussianNoise>
+          <gaussianNoise>0.03</gaussianNoise>
       </plugin>
      </sensor>

File: rotors_description/urdf/component_snippets.xacro (robot description, xacro)
@@ -17,5 +17,5 @@
 -->
 <robot xmlns:xacro="http://ros.org/wiki/xacro">
-  <xacro:property name="M_PI" value="3.14159265359" />
+  <xacro:property name="pi" value="3.14159265359" />
   <!-- Macro to add logging to a bag file. -->
   <xacro:macro name="bag_plugin_macro"
@@ -28,60 +28,6 @@
         <frameId>${namespace}/base_link</frameId>
         <rotorVelocitySlowdownSim>${rotor_velocity_slowdown_sim}</rotorVelocitySlowdownSim>
-	      <waitToRecordBag>${wait_to_record_bag}</waitToRecordBag>
+	<waitToRecordBag>${wait_to_record_bag}</waitToRecordBag>
       </plugin>
-    </gazebo>
-  </xacro:macro>
-<!-- Macro to add Hokuyo range sensor -->
-<xacro:macro name="hokuyo_lidar" params="namespace parent_link">
-    <link name="${namespace}/hokuyo_link">
-      <inertial>
-         <mass value="0.01" />
-         <inertia ixx="1e-6" ixy="0.0" ixz="0.0" iyy="1e-6" iyz="0.0" izz="1e-6" />
-      </inertial>
-      <visual name="visual">
-        <geometry>
-          <mesh filename="package://rotors_description/meshes/hokuyo.dae" />
-        </geometry>
-      </visual>
-     </link>
-     <joint name="laser" type="fixed">
-      <parent link="${parent_link}" />
-      <child link="${namespace}/hokuyo_link" />
-      <origin xyz="0 0 0.05" rpy="0 0 0" />
-    </joint>
-    <gazebo reference="${namespace}/hokuyo_link">
-    <sensor type="gpu_ray" name="head_hokuyo_sensor">
-      <pose>0 0 0 0 0 0</pose>
-      <visualize>false</visualize>
-      <update_rate>40</update_rate>
-      <ray>
-        <scan>
-          <horizontal>
-            <samples>720</samples>
-            <resolution>1</resolution>
-            <min_angle>-2.35619</min_angle>
-            <max_angle>2.35619</max_angle>
-          </horizontal>
-        </scan>
-        <range>
-          <min>0.10</min>
-          <max>30.0</max>
-          <resolution>0.01</resolution>
-        </range>
-        <noise>
-          <type>gaussian</type>
-          <!-- Noise parameters based on published spec for Hokuyo laser
-               achieving "+-30mm" accuracy at range < 10m.  A mean of 0.0m and
-               stddev of 0.01m will put 99.7% of samples within 0.03m of the true
-               reading. -->
-          <mean>0.0</mean>
-          <stddev>0.01</stddev>
-        </noise>
-      </ray>
-      <plugin name="gazebo_ros_head_hokuyo_controller" filename="libgazebo_ros_gpu_laser.so">
-        <topicName>/drone11/scan</topicName>
-        <frameName>hokuyo_link</frameName>
-      </plugin>
-    </sensor>
     </gazebo>
   </xacro:macro>
@@ -323,10 +269,10 @@
       <plugin name="mavlink_interface" filename="librotors_gazebo_mavlink_interface.so">
         <robotNamespace>${namespace}</robotNamespace>
-	      <mavlinkControlSubTopic>${mavlink_sub_topic}</mavlinkControlSubTopic>
+	<mavlinkControlSubTopic>${mavlink_sub_topic}</mavlinkControlSubTopic>
         <imuSubTopic>${imu_sub_topic}</imuSubTopic>
         <mavlinkHilSensorPubTopic>${mavlink_pub_topic}</mavlinkHilSensorPubTopic>
-	      <motorSpeedsPubTopic>${motors_speeds_pub_topic}</motorSpeedsPubTopic>
-	      <gpsUpdateFreq>${gps_update_freq}</gpsUpdateFreq> <!-- Frequency of HIL GPS messages [Hz] -->
-	      <rotorCount>${rotor_count}</rotorCount>
+	<motorSpeedsPubTopic>${motors_speeds_pub_topic}</motorSpeedsPubTopic>
+	<gpsUpdateFreq>${gps_update_freq}</gpsUpdateFreq> <!-- Frequency of HIL GPS messages [Hz] -->
+	<rotorCount>${rotor_count}</rotorCount>
         <!-- [Gauss] Below are the North, East, and Down components of the Earth's magnetic field at the reference location.
              The default reference location is Zurich (lat=+47.3667degN, lon=+8.5500degE, h=+500m, WGS84).
@@ -336,5 +282,5 @@
         <referenceMagEast>${reference_magnetic_field_east}</referenceMagEast>
         <referenceMagDown>${reference_magnetic_field_down}</referenceMagDown>
-	      <referenceLatitude>${reference_latitude}</referenceLatitude> <!-- the initial latitude [degrees [-90, 90]] -->
+	<referenceLatitude>${reference_latitude}</referenceLatitude> <!-- the initial latitude [degrees [-90, 90]] -->
         <referenceLongitude>${reference_longitude}</referenceLongitude> <!-- the initial longitude [degrees [-180, 180]] -->
         <referenceAltitude>${reference_altitude}</referenceAltitude> <!-- the initial altitude [m] -->
@@ -503,5 +449,5 @@
         <plugin filename="librotors_gazebo_gps_plugin.so" name="rotors_gazebo_gps${gps_suffix}_plugin">
           <robotNamespace>${namespace}</robotNamespace> <!-- (string, required): ros namespace in which the messages are published -->
-          <linkName>${namespace}/base_link</linkName> <!-- (string, required): name of the body which holds the GPS sensor -->
+          <linkName>${namespace}/gps${gps_suffix}_link</linkName> <!-- (string, required): name of the body which holds the GPS sensor -->
           <gpsTopic>${gps_topic}</gpsTopic> <!-- (string): name of the sensor output topic and prefix of service names (defaults to 'gps') -->
           <groundSpeedTopic>${ground_speed_topic}</groundSpeedTopic> <!-- (string): name of the ground speed output topic (defaults to 'ground_speed') -->
@@ -551,9 +497,40 @@
     </gazebo>
   </xacro:macro>
+  <!-- Macro to add an air pressure sensor. -->
+  <xacro:macro name="pressure_sensor_plugin_macro"
+    params="namespace pressure_sensor_suffix parent_link pressure_topic
+      mass_pressure_sensor reference_altitude pressure_variance *inertia
+      *origin">
+    <!-- Pressure sensor link -->
+    <link name="${namespace}/pressure_sensor${pressure_sensor_suffix}_link">
+      <inertial>
+        <xacro:insert_block name="inertia" />
+        <mass value="${mass_pressure_sensor}" />  <!-- [kg] -->
+        <origin xyz="0 0 0" rpy="0 0 0" />
+      </inertial>
+    </link>
+    <!-- Pressure sensor joint -->
+    <joint name="${namespace}/pressure_sensor${pressure_sensor_suffix}_joint" type="revolute">
+      <xacro:insert_block name="origin" />
+      <parent link="${parent_link}" />
+      <child link="${namespace}/pressure_sensor${pressure_sensor_suffix}_link" />
+      <limit upper="0" lower="0" effort="0" velocity="0" />
+    </joint>
+    <gazebo>
+      <plugin filename="librotors_gazebo_pressure_plugin.so" name="rotors_gazebo_pressure_sensor${pressure_sensor_suffix}_plugin">
+        <robotNamespace>${namespace}</robotNamespace> <!-- (string, required): ros namespace in which the messages are published -->
+        <linkName>${namespace}/pressure_sensor${pressure_sensor_suffix}_link</linkName> <!-- (string, required): name of the body which holds the pressure sensor -->
+        <pressureTopic>${pressure_topic}</pressureTopic> <!-- (string): name of the sensor output topic and prefix of service names (defaults to 'air_pressure') -->
+        <referenceAltitude>${reference_altitude}</referenceAltitude> <!-- the initial altitude [m] -->
+        <pressureVariance>${pressure_variance}</pressureVariance> <!-- the air pressure variance [Pa^2] -->
+      </plugin>
+    </gazebo>
+  </xacro:macro>
   <!-- Macro to add the wind plugin. -->
   <xacro:macro name="wind_plugin_macro"
     params="namespace xyz_offset wind_direction wind_force_mean
       wind_gust_direction wind_gust_duration wind_gust_start
-      wind_gust_force_mean wind_speed_mean">
+      wind_gust_force_mean wind_speed_mean use_custom_static_wind_field
+      custom_wind_field_path">
     <gazebo>
       <plugin filename="librotors_gazebo_wind_plugin.so" name="wind_plugin">
@@ -569,4 +546,6 @@
         <windGustForceMean>${wind_gust_force_mean}</windGustForceMean> <!-- [N] -->
         <windSpeedMean>${wind_speed_mean}</windSpeedMean> <!-- [m/s] -->
+        <useCustomStaticWindField>${use_custom_static_wind_field}</useCustomStaticWindField>
+        <customWindFieldPath>${custom_wind_field_path}</customWindFieldPath> <!-- from ~/.ros -->
       </plugin>
     </gazebo>
@@ -886,8 +865,17 @@
     </xacro:magnetometer_plugin_macro>
   </xacro:macro>
-  <!-- DEFAULT VALUES OF REFERENCES -->
-  <!--reference_latitude="47.3667"
-      reference_longitude="8.5500"
-      reference_altitude="500.0" -->
+  <xacro:macro name="default_pressure_sensor" params="namespace parent_link">
+    <xacro:pressure_sensor_plugin_macro
+      namespace="${namespace}"
+      pressure_sensor_suffix=""
+      parent_link="${parent_link}"
+      pressure_topic="air_pressure"
+      mass_pressure_sensor="0.015"
+      reference_altitude="500.0"
+      pressure_variance="0.0">
+      <inertia ixx="0.00001" ixy="0.0" ixz="0.0" iyy="0.00001" iyz="0.0" izz="0.00001" />
+      <origin xyz="0 0 0" rpy="0 0 0" />
+    </xacro:pressure_sensor_plugin_macro>
+  </xacro:macro>
   <xacro:macro name="default_mavlink_interface" params="namespace imu_sub_topic rotor_count">
     <xacro:mavlink_interface_macro
@@ -902,7 +890,7 @@
       reference_magnetic_field_east="0.00797"
       reference_magnetic_field_down="0.42817"
-      reference_latitude="49.9"
-      reference_longitude="8.9"
-      reference_altitude="0.0">
+      reference_latitude="47.3667"
+      reference_longitude="8.5500"
+      reference_altitude="500.0">
     </xacro:mavlink_interface_macro>
   </xacro:macro>

File: rotors_description/urdf/firefly_base.xacro (robot description, xacro)
@@ -16,5 +16,6 @@
   limitations under the License.
 -->
-<robot name="firefly" xmlns:xacro="http://ros.org/wiki/xacro">
+<robot name="firefly"
+  xmlns:xacro="http://ros.org/wiki/xacro">
   <xacro:include filename="$(find rotors_description)/urdf/component_snippets.xacro" />
   <xacro:include filename="$(find rotors_description)/urdf/component_mbzirc.xacro" />
@@ -37,11 +38,16 @@
     <xacro:gazebo_tf_plugin_macro namespace="${namespace}"/>
   </xacro:if>
+  <xacro:thermal_camera_macro namespace="${namespace}" parent_link="${namespace}/base_link" camera_suffix="unique">
+  </xacro:thermal_camera_macro>
+  <!-- Adding thermal camera looking down -->
+  <xacro:thermal_camera_down_macro namespace="${namespace}" parent_link="${namespace}/base_link" camera_suffix="unique">
+  </xacro:thermal_camera_down_macro>
+  <xacro:ouster_lidar namespace="${namespace}" parent_link="${namespace}/base_link">
+  </xacro:ouster_lidar>
+  <xacro:gps_fix_macro namespace="${namespace}" parent_link="${namespace}/base_link">
+  </xacro:gps_fix_macro>
   <xacro:if value="$(arg enable_logging)">
     <!-- Instantiate a logger -->
-    <xacro:bag_plugin_macro
-      namespace="${namespace}"
-      bag_file="$(arg log_file)"
-      rotor_velocity_slowdown_sim="${rotor_velocity_slowdown_sim}"
-      wait_to_record_bag="$(arg wait_to_record_bag)" />
+    <xacro:bag_plugin_macro namespace="${namespace}" bag_file="$(arg log_file)" rotor_velocity_slowdown_sim="${rotor_velocity_slowdown_sim}" wait_to_record_bag="$(arg wait_to_record_bag)" />
   </xacro:if>
 </robot>
